File: prototype/teensy_sync_rev1.brd (EAGLE design)
At the start: 57.1 x 41.3 mm, 15 parts, among them U1 MPU-6000QFN-24

Commit message: Modified board headers. F3 header has now been integrated in to C31 header. Old F3 header now serves as communication line breakout.
Connections:
- removed net C31_IO2: J2.5, U$2.7
- removed net C31_IO3: J2.4, U$2.9
- removed net F3_I0: J1.1, U$2.15/A1
- removed net F3_O1: J1.2, U$2.16/A2
- removed net F3_RX: J1.4, U$2.1
- removed net F3_TX: J1.3, U$2.0
- new net C31_IO2_RX: J2.5, U$2.1
- new net C31_IO3_TX: J2.4, U$2.0
- net 3.3V: now also J1.2
- net C32_IO2: now also U$2.6; no longer U$2.8
- net C32_IO3: now also U$2.7; no longer U$2.10
- net GND: now also J1.1; no longer J1.5, J1.6
- net IMU1_CS: now also J1.3, U$2.17/A3; no longer U$2.14/A0
- net MISO: now also J1.6
- net MOSI: now also J1.5
- net SCK: now also J1.4
- net SCL: now also J1.8
- net SDA: now also J1.7
Routing:
- net F3_TX: track 44.2 -> 0.00 mm
- net F3_RX: track 39.1 -> 0.00 mm
- net SCL: track 9.59 -> 43.5 mm
- net SDA: track 15.0 -> 42.3 mm, vias 0 -> 1
- net C31_IO3_TX: track 0.00 -> 22.2 mm
- net 3.3V: track 69.8 -> 87.3 mm, vias 2 -> 5
- net C31_IO2_RX: track 0.00 -> 16.2 mm
- net F3_O1: track 11.6 -> 0.00 mm
- net IMU1_CS: track 41.3 -> 52.4 mm
- net C31_IO3: track 10.1 -> 0.00 mm
- net F3_I0: track 9.62 -> 0.00 mm
- net SCK: track 47.0 -> 55.8 mm
- net MISO: track 63.7 -> 71.7 mm, vias 1 -> 0
- net C32_IO3: track 14.4 -> 6.64 mm
- net C31_IO2: track 7.19 -> 0.00 mm
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