File: prototype/teensy_sync_rev1.sch (EAGLE design)
At the start: 15 parts, among them U1 MPU-6000QFN-24

Commit message: Modified board headers. F3 header has now been integrated in to C31 header. Old F3 header now serves as communication line breakout.
Connections:
- removed net C31_IO2: J2.5, U$2.7/RX3
- removed net C31_IO3: J2.4, U$2.9/RX2/PWM
- removed net F3_I0: J1.1, U$2.15/A1/T
- removed net F3_O1: J1.2, U$2.16/A2/T
- removed net F3_RX: J1.4, U$2.1/TX1/T
- removed net F3_TX: J1.3, U$2.0/RX1/T
- new net C31_IO2_RX: J2.5, U$2.1/TX1/T
- new net C31_IO3_TX: J2.4, U$2.0/RX1/T
- net 3.3V: now also J1.2
- net C32_IO2: now also U$2.6/PWM; no longer U$2.8/TX3
- net C32_IO3: now also U$2.7/RX3; no longer U$2.10/TX2/PWM
- net GND: now also J1.1; no longer J1.5, J1.6
- net IMU1_CS: now also J1.3, U$2.17/A3/T; no longer U$2.14/A1
- net MISO: now also J1.6
- net MOSI: now also J1.5
- net SCK: now also J1.4
- net SCL: now also J1.8
- net SDA: now also J1.7
