File: prototype/teensy_sync.brd (EAGLE design)
At the start: 57.1 x 41.3 mm, 15 parts, among them U1 MPU-6000QFN-24

Commit message: Updated brd and sch file to reflect prototype boards ordered.
Parts:
- added JP2: JUMPER-SMT_3_NO_SILK, SparkFun-Jumpers:SMT-JUMPER_3_NO_SILK
- C6: value (none) -> 0.1uF
- U$2: value TEENSY_3.1_DIL -> TEENSY_3.2
Connections:
- removed net AGND: U$2.AGND
- new net C32_IO3_T: JP2.3, U$2.7
- net C31_IO3_TX: now also JP2.1
- net C32_IO3: now also JP2.2; no longer U$2.7
- net GND: now also U$2.AGND
- net IMU1_DIO4: now also U$2.21/A7
Routing:
- net IMU1_DIO4: track 0.00 -> 32.3 mm, vias 0 -> 1
- net IMU1_CS: track 52.4 -> 58.7 mm, vias 0 -> 1
- net 3.3V: track 87.3 -> 83.6 mm, vias 5 -> 2
- net IMU1_DIO1: track 20.5 -> 23.4 mm, vias 1 -> 0
- net MISO: track 71.7 -> 74.4 mm, vias 0 -> 2
- net C32_IO3_T: track 0.00 -> 2.56 mm
- net C32_IO3: track 6.64 -> 8.86 mm
- net C31_IO3_TX: track 22.2 -> 24.4 mm
- net SCK: track 55.8 -> 57.0 mm, vias 1 -> 0
- net GND: track 18.3 -> 17.4 mm
Other:
- board text added: "DEP"
- board text added: "IND"
- board text added: "svis_pcb"
- board text removed: "Camera Sync Board Rev1"
